Commit message: add gazebo control

File: description/robot.urdf.xacro (robot description, xacro)
@@ -2,3 +2,4 @@
 <robot xmlns:xacro="http://www.ros.org/wiki/xacro"  name="racer_bot">
 <xacro:include filename="robot_core.xacro" />
+<xacro:include filename="gazebo_control.xacro"/>
 </robot>

File: description/robot_core.xacro (robot description, xacro)
@@ -40,4 +40,7 @@
         </xacro:inertial_box>
     </link>
+    <gazebo reference="chassis">
+        <material>Gazebo/White</material>
+    </gazebo>
 <!-- FRONT BUMPER-->
     <joint name="bumper_joint" type = "fixed">
@@ -66,5 +69,5 @@
         <parent link="body"/>
         <child link="rear_left_axel_link"/>
-        <origin xyz="-0.156 0.058 0" rpy="${pi/2} 0 0 "/>
+        <origin xyz="-0.156 0.059 0" rpy="-${pi/2} 0 0 "/>
     </joint>
     <link name="rear_left_axel_link">
@@ -84,9 +87,12 @@
         </xacro:inertial_cylinder>
     </link>
+    <gazebo reference="rear_left_axel_link">
+        <material>Gazebo/Orange</material>
+    </gazebo>
 <!-- REAR RIGHT WHEEL AXEL -->
     <joint name="rear_right_axel_joint" type="fixed">
         <parent link="body"/>
         <child link="rear_right_axel_link"/>
-        <origin xyz="-0.15 -0.058 0" rpy="${pi/2} 0 0 "/>
+        <origin xyz="-0.15 -0.059 0" rpy="${pi/2} 0 0 "/>
     </joint>
     <link name="rear_right_axel_link">
@@ -106,9 +112,12 @@
         </xacro:inertial_cylinder>
     </link>
+    <gazebo reference="rear_right_axel_link">
+        <material>Gazebo/Orange</material>
+    </gazebo>
 <!-- FRONT LEFT WHEEL AXEL -->
     <joint name="front_left_axel_joint" type="fixed">
         <parent link="body"/>
         <child link="front_left_axel_link"/>
-        <origin xyz="0.145 0.058 0" rpy="-${pi/2} 0 0"/>
+        <origin xyz="0.145 0.059 0" rpy="-${pi/2} 0 0"/>
     </joint>
     <link name="front_left_axel_link">
@@ -128,9 +137,12 @@
         </xacro:inertial_cylinder>
     </link>
+    <gazebo reference="front_left_axel_link">
+        <material>Gazebo/Orange</material>
+    </gazebo>
 <!-- FRONT RIGHT WHEEL AXEL -->
     <joint name="front_right_axel_joint" type="fixed">
         <parent link="body"/>
         <child link="front_right_axel_link"/>
-        <origin xyz="0.145 -0.058 0" rpy="${pi/2} 0 0"/>
+        <origin xyz="0.145 -0.059 0" rpy="${pi/2} 0 0"/>
     </joint>
     <link name="front_right_axel_link">
@@ -150,4 +162,7 @@
         </xacro:inertial_cylinder>
     </link>
+    <gazebo reference="front_right_axel_link">
+        <material>Gazebo/Orange</material>
+    </gazebo>
 <!-- FRONT LEFT WHEEL -->
     <joint name="front_left_wheel_joint" type="continuous">
@@ -173,4 +188,9 @@
         </xacro:inertial_cylinder>
     </link>
+    <gazebo reference="front_left_wheel">
+        <material>Gazebo/Blue</material>
+        <mu1 value="0.001"/>
+        <mu2 value="0.001"/>
+    </gazebo>
 <!-- FRONT RIGHT WHEEL -->
     <joint name="front_right_wheel_joint" type="continuous">
@@ -196,9 +216,14 @@
         </xacro:inertial_cylinder>
     </link>
+    <gazebo reference="front_right_wheel">
+        <material>Gazebo/Blue</material>
+        <mu1 value="0.001"/>
+        <mu2 value="0.001"/>
+    </gazebo>
 <!-- BACK LEFT WHEEL -->
     <joint name="rear_left_wheel_joint" type="continuous">
         <parent link="rear_left_axel_link"/>
         <child link="rear_left_wheel"/>
-        <origin xyz="0 0 -0.044" rpy="0 0 0"/>
+        <origin xyz="0 0 0.044" rpy="0 0 0"/>
         <axis xyz="0 0 1"/>
     </joint>
@@ -219,4 +244,7 @@
         </xacro:inertial_cylinder>
     </link>
+    <gazebo reference="rear_left_wheel">
+        <material>Gazebo/Blue</material>
+    </gazebo>
 <!-- BACK RIGHT WHEEL -->
     <joint name="rear_right_wheel_joint" type="continuous">
@@ -242,3 +270,6 @@
         </xacro:inertial_cylinder>
     </link>
+    <gazebo reference="rear_right_wheel">
+        <material>Gazebo/Blue</material>
+    </gazebo>
 </robot>

Commit message: add lidar to model

File: description/robot.urdf.xacro (robot description, xacro)
@@ -3,3 +3,4 @@
 <xacro:include filename="robot_core.xacro" />
 <xacro:include filename="gazebo_control.xacro"/>
+<xacro:include filename="lidar.xacro"/>
 </robot>

File: description/robot_core.xacro (robot description, xacro)
@@ -14,14 +14,17 @@
         <color rgba="0 0 0 1"/>
     </material>
+    <material name="red">
+        <color rgba="1 0 0 1"/>
+    </material>
 <!-- BASE LINK-->
     <link name="base_link">
     </link>
 <!-- CAHSSIS LINK-->
-    <joint name="body_joint" type = "fixed">
+    <joint name="chassis_joint" type = "fixed">
         <parent link ="base_link" />
-        <child link="body"/>
+        <child link="chassis"/>
         <origin xyz="0.15 0 0"/>
     </joint>
-    <link name="body">
+    <link name="chassis">
         <visual>
             <geometry>
@@ -45,5 +48,5 @@
 <!-- FRONT BUMPER-->
     <joint name="bumper_joint" type = "fixed">
-        <parent link ="body" />
+        <parent link ="chassis" />
         <child link="front_bumper"/>
         <origin xyz="0.209 0 0"/>
@@ -52,5 +55,5 @@
         <visual>
             <geometry>
-                <box size="0.01 0.265 0.057"/>
+                <box size="0.01 0.265 0.0285"/>
             </geometry>
             <material name="white"/>
@@ -67,5 +70,5 @@
 <!--REAR LEFT WHEEL AXEL -->
     <joint name="rear_left_axel_joint" type="fixed">
-        <parent link="body"/>
+        <parent link="chassis"/>
         <child link="rear_left_axel_link"/>
         <origin xyz="-0.156 0.059 0" rpy="-${pi/2} 0 0 "/>
@@ -92,5 +95,5 @@
 <!-- REAR RIGHT WHEEL AXEL -->
     <joint name="rear_right_axel_joint" type="fixed">
-        <parent link="body"/>
+        <parent link="chassis"/>
         <child link="rear_right_axel_link"/>
         <origin xyz="-0.15 -0.059 0" rpy="${pi/2} 0 0 "/>
@@ -117,5 +120,5 @@
 <!-- FRONT LEFT WHEEL AXEL -->
     <joint name="front_left_axel_joint" type="fixed">
-        <parent link="body"/>
+        <parent link="chassis"/>
         <child link="front_left_axel_link"/>
         <origin xyz="0.145 0.059 0" rpy="-${pi/2} 0 0"/>
@@ -142,5 +145,5 @@
 <!-- FRONT RIGHT WHEEL AXEL -->
     <joint name="front_right_axel_joint" type="fixed">
-        <parent link="body"/>
+        <parent link="chassis"/>
         <child link="front_right_axel_link"/>
         <origin xyz="0.145 -0.059 0" rpy="${pi/2} 0 0"/>
